Commit message: sabuvis

File: uuv_gazebo_plugins/uuv_gazebo_ros_plugins/urdf/fin_snippets.xacro (robot description, xacro)
@@ -73,8 +73,12 @@
             drag_constant
             current_velocity_topic">
+            <!-- *origin_link -->
     <joint name="${namespace}/fin${fin_id}_joint" type="revolute">
+    <!-- <joint name="${namespace}/fin${fin_id}_joint" type="fixed"> -->
+        <!-- <axis xyz="0 0 0"/> -->
         <limit effort="0" lower="${min_joint_limit}" upper="${max_joint_limit}" velocity="0"/>
+        <!-- <limit effort="-1" lower="${min_joint_limit}" upper="${max_joint_limit}" velocity="-1"/> -->
         <xacro:insert_block name="origin"/>
-        <axis xyz="0 0 1"/>
+        <axis xyz="0 1 0"/>
         <parent link="${parent_link}" />
         <child link="${namespace}/fin${fin_id}" />
@@ -82,8 +86,12 @@
     <link name="${namespace}/fin${fin_id}">
       <xacro:no_inertial />
+      <!-- <xacro:box_inertial x="0" y="0" z="0" mass="0.001">
+        <origin xyz="0 0 0" rpy="0 0 0"/>
+      </xacro:box_inertial> -->
       <visual>
-        <origin xyz="0 0 0" rpy="0 0 0" />
+        <origin xyz="0 0 0" rpy="${3.14*fin_id} 0 0" />
+        <!-- <xacro:insert_block name="origin_link"/> -->
         <geometry>
-          <mesh filename="${mesh_filename}" scale="1 1 1"/>
+          <mesh filename="${mesh_filename}" scale="0.001 0.001 0.001"/>
         </geometry>
       </visual>

File: uuv_gazebo_plugins/uuv_gazebo_ros_plugins/urdf/thruster_snippets.xacro (robot description, xacro)
@@ -84,4 +84,5 @@
     <link name="${namespace}/thruster_${thruster_id}">
       <xacro:box_inertial x="0" y="0" z="0" mass="0.001">
+      <!-- <xacro:box_inertial x="0" y="0" z="0" mass="1.0"> -->
         <origin xyz="0 0 0" rpy="0 0 0"/>
       </xacro:box_inertial>
@@ -89,5 +90,6 @@
         <origin rpy="0 0 0" xyz="0 0 0"/>
         <geometry>
-          <mesh filename="${mesh_filename}" scale="1 1 1"/>
+          <!-- <mesh filename="${mesh_filename}" scale="1 1 1"/> -->
+          <mesh filename="${mesh_filename}" scale="0.5 0.5 0.5"/>
         </geometry>
       </visual>

Commit message: update

File: uuv_gazebo_plugins/uuv_gazebo_ros_plugins/urdf/fin_snippets.xacro (robot description, xacro)
@@ -65,5 +65,5 @@
             parent_link
             fin_id
-            *origin
+            scale
             min_joint_limit
             max_joint_limit
@@ -72,6 +72,8 @@
             lift_constant
             drag_constant
-            current_velocity_topic">
-            <!-- *origin_link -->
+            current_velocity_topic
+            visual_rpy
+            *origin">
+            <!-- **origin_link -->
     <joint name="${namespace}/fin${fin_id}_joint" type="revolute">
     <!-- <joint name="${namespace}/fin${fin_id}_joint" type="fixed"> -->
@@ -80,5 +82,6 @@
         <!-- <limit effort="-1" lower="${min_joint_limit}" upper="${max_joint_limit}" velocity="-1"/> -->
         <xacro:insert_block name="origin"/>
-        <axis xyz="0 1 0"/>
+        <!-- <axis xyz="0 1 0"/> -->
+        <axis xyz="0 0 1"/>
         <parent link="${parent_link}" />
         <child link="${namespace}/fin${fin_id}" />
@@ -90,8 +93,12 @@
       </xacro:box_inertial> -->
       <visual>
-        <origin xyz="0 0 0" rpy="${3.14*fin_id} 0 0" />
+        <!-- <origin xyz="0 0 0" rpy="${3.14*fin_id} 0 0" /> -->
+        <!-- <origin xyz="0 0 0" rpy="0 ${-3.14/2} ${3.14/2}" /> -->
+        <origin xyz="0 0 0" rpy="${visual_rpy}" />
         <!-- <xacro:insert_block name="origin_link"/> -->
         <geometry>
-          <mesh filename="${mesh_filename}" scale="0.001 0.001 0.001"/>
+          <!-- <mesh filename="${mesh_filename}" scale="0.001 0.001 0.001"/> -->
+          <!-- <mesh filename="${mesh_filename}" scale="1.0 1.0 1.0"/> -->
+          <mesh filename="${mesh_filename}" scale="${scale}"/>
         </geometry>
       </visual>

File: uuv_gazebo_plugins/uuv_gazebo_ros_plugins/urdf/thruster_snippets.xacro (robot description, xacro)
@@ -87,11 +87,10 @@
         <origin xyz="0 0 0" rpy="0 0 0"/>
       </xacro:box_inertial>
-      <visual>
+      <!-- <visual>
         <origin rpy="0 0 0" xyz="0 0 0"/>
         <geometry>
-          <!-- <mesh filename="${mesh_filename}" scale="1 1 1"/> -->
           <mesh filename="${mesh_filename}" scale="0.5 0.5 0.5"/>
         </geometry>
-      </visual>
+      </visual> -->
       <collision>
         <!-- todo: gazebo needs a collision volume or it will ignore the pose of

File: uuv_sensor_plugins/uuv_sensor_ros_plugins/urdf/camera_snippets.xacro (robot description, xacro)
@@ -138,4 +138,8 @@
           <pointCloudCutoff>10.0</pointCloudCutoff>
         </plugin>
+        <!-- <plugin name="GstCameraPlugin" filename="libgazebo_gst_camera_plugin.so">
+          <robotNamespace>"${namespace}"</robotNamespace>
+          <udpPort>5600</udpPort>
+        </plugin> -->
       </sensor>
     </gazebo>

File: uuv_sensor_plugins/uuv_sensor_ros_plugins/urdf/pose_3d_snippets.xacro (robot description, xacro)
@@ -64,5 +64,5 @@
       parent_link="${parent_link}"
       topic="pose_gt"
-      update_rate="20"
+      update_rate="100"
       noise_sigma="0.0"
       noise_amplitude="0.0"

File: uuv_sensor_plugins/uuv_sensor_ros_plugins/urdf/pressure_snippets.xacro (robot description, xacro)
@@ -32,5 +32,5 @@
       noise_sigma="3.0"
       noise_amplitude="0.0"
-      estimateDepth="false"
+      estimateDepth="true"
       standardPressure="101.325"
       kPaPerM="9.80638">

File: uuv_sensor_plugins/uuv_sensor_ros_plugins/urdf/sonar_snippets.xacro (robot description, xacro)
@@ -193,7 +193,11 @@
           </save>
         </camera>
-	    <plugin filename="libimage_sonar_ros_plugin.so" name="forward_sonar${suffix}_controller">
-		  <topicName>${topic}</topicName>
+        <plugin filename="libimage_sonar_ros_plugin.so" name="forward_sonar${suffix}_controller">
+          <topicName>${topic}</topicName>
           <frameName>forward_sonar${suffix}_optical_frame</frameName>
+          <clip>
+            <near>0.1</near>
+            <far>17</far>
+          </clip>
         </plugin>
         <always_on>true</always_on>

Commit message: fins collision

File: uuv_gazebo_plugins/uuv_gazebo_ros_plugins/urdf/fin_snippets.xacro (robot description, xacro)
@@ -88,8 +88,8 @@
     </joint>
     <link name="${namespace}/fin${fin_id}">
-      <xacro:no_inertial />
-      <!-- <xacro:box_inertial x="0" y="0" z="0" mass="0.001">
+      <!-- <xacro:no_inertial /> -->
+      <xacro:box_inertial x="0.01" y="0.01" z="0.01" mass="0.01">
         <origin xyz="0 0 0" rpy="0 0 0"/>
-      </xacro:box_inertial> -->
+      </xacro:box_inertial>
       <visual>
         <!-- <origin xyz="0 0 0" rpy="${3.14*fin_id} 0 0" /> -->
@@ -103,4 +103,10 @@
         </geometry>
       </visual>
+      <collision>
+        <origin xyz="0 0 0" rpy="${visual_rpy}" />
+        <geometry>
+          <mesh filename="${mesh_filename}" scale="${scale}"/>
+        </geometry>
+      </collision>
     </link>
     <gazebo>

Commit message: fins_collision

File: uuv_gazebo_plugins/uuv_gazebo_ros_plugins/urdf/fin_snippets.xacro (robot description, xacro)
@@ -104,7 +104,8 @@
       </visual>
       <collision>
-        <origin xyz="0 0 0" rpy="${visual_rpy}" />
+        <origin xyz="-0.2 0 ${0.3 * (fin_id-0.5)}" rpy="${visual_rpy}" />
         <geometry>
-          <mesh filename="${mesh_filename}" scale="${scale}"/>
+          <!-- <mesh filename="${mesh_filename}" scale="${scale}"/> -->
+          <box size="0.2 0.2 0.025" />
         </geometry>
       </collision>
